File: RailroadShield.brd (EAGLE design)
At the start: 99.6 x 78.7 mm, 61 parts, among them J1 5520250-3, J2 5520250-3, J3 5520250-3, J4 5520426-4, J5 5520426-4, J6 KK-156-5, J7 KK-156-5, J8 MSTB-02, Q1 PMBT2222, U1 LM393M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

Commit message: 2.4
Parts:
- added F1: PTCPTH, SparkFun:PTC
- D1, D2: value 1N4448WT -> BAV199; device MCP:SOT23-3 -> diode:SOT23
- JP2: value ShieldGnd -> CMRI Shield
- LED5: value DCC -> Yellow
- LED6: value Loconet -> Blue
- SV1, SV2: value (none) -> 929850-01-15
- Y1: value 16Mhz -> 16Mhz 81-CSTLS16M0X53-B0
- moved C2 9.20 mm to (58.4, 30.5), turned to 0 degrees
- moved RN2 7.94 mm to (19.8, 50.8)
- moved Y1 5.61 mm to (47.0, 31.8)
- moved J6 5.59 mm to (38.1, 5.08)
- moved R13 5.34 mm to (57.1, 25.4)
- moved J7 5.09 mm to (61.0, 5.08)
- moved U2 5.09 mm to (48.3, 22.9)
- moved C3 5.08 mm to (66.0, 32.0)
- moved JP2 5.08 mm to (73.7, 7.37)
- moved R11 5.05 mm to (59.7, 25.4)
- moved U3 4.83 mm to (66.0, 25.4)
- moved LED6 4.35 mm to (95.2, 72.4)
- moved R9 3.39 mm to (95.2, 76.2)
- moved L1 3.31 mm to (75.7, 27.9)
- moved LED5 2.34 mm to (2.54, 73.7), turned to 0 degrees
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Connections:
- removed net TERM-PWR: JP1.1, U7.1
- new net N$20: JP1.2, R10.2, U7.4
- new net N$21: F1.P$2, U$1.VIN
- net LOCONET: now also JP1.1; no longer R10.2, U7.4
- net V+: now also F1.P$1, U7.1; no longer JP1.2, U$1.VIN
Routing:
- net V+: track 219.6 -> 127.7 mm
- net LNRX: track 124.0 -> 74.7 mm, vias 1 -> 2
- net VCC: track 233.0 -> 265.1 mm, vias 9 -> 5
- net TERM-PWR: track 30.9 -> 0.00 mm, vias 2 -> 0
- net O-RESB: track 22.3 -> 52.6 mm
- net N$20: track 0.00 -> 28.8 mm
- net N$7: track 76.0 -> 54.3 mm, vias 2 -> 0
- net GND: track 107.6 -> 87.6 mm, vias 11 -> 10
- net N$8: track 70.4 -> 51.7 mm, vias 2 -> 3
- net CAN-L: track 42.1 -> 59.3 mm
- net N$9: track 65.0 -> 77.7 mm
- net NCERX: track 63.0 -> 50.5 mm
- net N$21: track 0.00 -> 12.1 mm
- net N$19: track 75.8 -> 64.6 mm, vias 1 -> 2
- net MISO: track 52.5 -> 63.4 mm
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Other:
- board text added: "Fixed: aligned parts to grid"
- board text added: "Fixed: clearance problems"
- board text added: "Fixed: component labeling problems"
- board text added: "Ground"
- board text added: "Rev. 2.4"
- board text added: "v2.4"
- board text removed: "Rev. 2.3"

Commit message: 2.5
Parts:
- added U$2: OSHW-LOGOM, SparkFun:OSHW-LOGO-M
Other:
- board text added: "Fixed: Added Open Source Hardware Label"
- board text added: "Hardware"
- board text added: "Open Source"
- board text added: "Rev. 2.5"
- board text removed: "Fixed: aligned parts to grid"
- board text removed: "Fixed: clearance problems"
- board text removed: "Fixed: component labeling problems"
- board text removed: "Rev. 2.4"
Changed lines of the file:
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@@
 <layer number="97" name="Info" color="7" fill="1" visible="no" active="no"/>
 <layer number="98" name="Guide" color="6" fill="1" visible="no" active="no"/>
+<layer number="99" name="Anatomie" color="7" fill="1" visible="no" active="no"/>
 <layer number="101" name="Bemassung" color="7" fill="1" visible="yes" active="yes"/>
 <layer number="2" name="Route2" color="1" fill="3" visible="no" active="no"/>
@@
 <layer number="109" name="fp9" color="7" fill="1" visible="no" active="no"/>
 <layer number="110" name="fp0" color="7" fill="1" visible="no" active="no"/>
+<layer number="111" name="bdokum" color="7" fill="1" visible="no" active="no"/>
 <layer number="116" name="Patch_BOT" color="9" fill="4" visible="no" active="no"/>
 <layer number="121" name="_tsilk" color="7" fill="1" visible="no" active="no"/>
@@
 <layer number="123" name="tTestmark" color="7" fill="1" visible="no" active="no"/>
 <layer number="124" name="bTestmark" color="7" fill="1" visible="no" active="no"/>
+<layer number="125" name="_tNames" color="7" fill="1" visible="no" active="no"/>
+<layer number="126" name="_bNames" color="7" fill="1" visible="no" active="no"/>
 <layer number="131" name="tAdjust" color="7" fill="1" visible="no" active="no"/>
 <layer number="132" name="bAdjust" color="7" fill="1" visible="no" active="no"/>
@@
 <layer number="209" name="209bmp" color="7" fill="1" visible="no" active="no"/>
 <layer number="210" name="210bmp" color="7" fill="1" visible="no" active="no"/>
+<layer number="211" name="211bmp" color="7" fill="1" visible="no" active="no"/>
+<layer number="212" name="212bmp" color="7" fill="1" visible="no" active="no"/>
+<layer number="213" name="213bmp" color="7" fill="1" visible="no" active="no"/>
+<layer number="214" name="214bmp" color="7" fill="1" visible="no" active="no"/>
+<layer number="215" name="215bmp" color="7" fill="1" visible="no" active="no"/>
+<layer number="216" name="216bmp" color="7" fill="1" visible="no" active="no"/>
+<layer number="217" name="217bmp" color="18" fill="1" visible="no" active="no"/>
+<layer number="218" name="218bmp" color="19" fill="1" visible="no" active="no"/>
+<layer number="219" name="219bmp" color="20" fill="1" visible="no" active="no"/>
+<layer number="220" name="220bmp" color="21" fill="1" visible="no" active="no"/>
+<layer number="221" name="221bmp" color="22" fill="1" visible="no" active="no"/>
+<layer number="222" name="222bmp" color="23" fill="1" visible="no" active="no"/>
+<layer number="223" name="223bmp" color="24" fill="1" visible="no" active="no"/>
+<layer number="224" name="224bmp" color="25" fill="1" visible="no" active="no"/>
 <layer number="250" name="Descript" color="3" fill="1" visible="no" active="no"/>
 <layer number="251" name="SMDround" color="12" fill="11" visible="no" active="no"/>
@@
 <wire x1="33.274" y1="42.926" x2="23.622" y2="42.926" width="0.254" layer="48"/>
 <wire x1="23.622" y1="42.926" x2="23.622" y2="43.434" width="0.254" layer="48"/>
-<wire x1="22.606" y1="10.414" x2="1.27" y2="10.414" width="0" layer="48"/>
-<wire x1="17.018" y1="10.16" x2="17.018" y2="0.762" width="0" layer="48"/>
+<wire x1="22.606" y1="10.414" x2="17.272" y2="10.414" width="0" layer="48"/>
+<wire x1="17.272" y1="10.414" x2="1.27" y2="10.414" width="0" layer="48"/>
+<wire x1="26.67" y1="9.906" x2="26.67" y2="1.016" width="0" layer="48"/>
+<wire x1="26.67" y1="1.016" x2="26.67" y2="0.508" width="0" layer="48"/>
 <wire x1="41.91" y1="53.848" x2="41.91" y2="52.578" width="0.3048" layer="48"/>
 <wire x1="70.866" y1="14.478" x2="70.866" y2="15.24" width="0.254" layer="48"/>
@@
 <wire x1="41.91" y1="55.372" x2="41.91" y2="55.118" width="0.3048" layer="48"/>
 <wire x1="39.624" y1="55.372" x2="40.005" y2="55.118" width="0.3048" layer="48"/>
+<wire x1="22.606" y1="10.414" x2="26.67" y2="10.414" width="0" layer="48"/>
+<wire x1="26.67" y1="10.414" x2="26.67" y2="9.906" width="0" layer="48"/>
 <text x="100.9015" y="59.1185" size="1.27" layer="48" font="vector" rot="R90">Loconet</text>
 <text x="97.155" y="33.274" size="0.8128" layer="48" font="vector" rot="R270">Component Side</text>
 <text x="96.52" y="6.096" size="0.8128" layer="26" font="vector" rot="MR90">Solder Side</text>
-<text x="88.011" y="37.211" size="0.8128" layer="48" font="vector">John Plocher</text>
+<text x="27.813" y="1.143" size="0.8128" layer="48" font="vector" rot="R90">John Plocher</text>
 <text x="52.959" y="34.163" size="0.8128" layer="48" font="vector">2011.07</text>
-<text x="81.534" y="35.306" size="1.016" layer="48" font="vector" rot="R180">Rev. 2.4</text>
+<text x="81.534" y="35.306" size="1.016" layer="48" font="vector" rot="R180">Rev. 2.5</text>
 <text x="53.086" y="36.068" size="2.54" layer="48" font="vector" ratio="15">RailroadShield</text>
 <text x="101.1555" y="44.0055" size="1.27" layer="48" font="vector" rot="R90">Loconet</text>
@@
 <text x="36.068" y="10.16" size="1.27" layer="48" font="vector">+OUT-</text>
 <text x="1.8034" y="16.6624" size="2.1844" layer="48" font="vector" ratio="15">NCE</text>
-<text x="19.05" y="4.826" size="2.1844" layer="48" font="vector" ratio="15">C/MRI</text>
+<text x="50.546" y="0.762" size="2.1844" layer="48" font="vector" ratio="15" rot="R90">C/MRI</text>
 <text x="64.262" y="51.308" size="1.27" layer="26" font="vector" ratio="15" rot="MR180">.com</text>
 <text x="90.678" y="57.15" size="1.27" layer="26" font="vector" ratio="15" rot="MR0">www.</text>
@@
 <text x="33.528" y="63.754" size="0.8128" layer="48" font="vector" ratio="15">Made in the PCR, Coast Division, NMRA</text>
 <text x="98.3615" y="2.3495" size="1.016" layer="48" font="vector" rot="R90">seeed: 31126</text>
-<text x="103.886" y="0" size="0.6096" layer="49" rot="R90">Fixed: component labeling problems</text>
-<text x="105.156" y="0" size="0.6096" layer="49" rot="R90">Fixed: clearance problems</text>
-<text x="106.68" y="0" size="0.6096" layer="49" rot="R90">Fixed: aligned parts to grid</text>
+<text x="103.886" y="0" size="0.6096" layer="49" rot="R90">Fixed: Added Open Source Hardware Label</text>
 <text x="75.438" y="9.906" size="0.8128" layer="48" rot="R180">Ground</text>
 <text x="77.47" y="39.624" size="3.81" layer="26" font="vector" ratio="20" rot="MR180">v2.4</text>
+<text x="16.002" y="8.89" size="1.016" layer="48">Open Source</text>
+<text x="16.51" y="2.286" size="1.016" layer="48">Hardware</text>
 </plain>
 <attributes>
@@
 <element name="J6" library="MCP" package="KK-156-5" value="KK-156-5" x="38.1" y="5.08" smashed="yes" rot="R180">
 <attribute name="NAME" x="30.861" y="8.134" size="1.27" layer="25"/>
-<attribute name="VALUE" x="49.27" y="9.525" size="1.27" layer="27" rot="R270"/>
+<attribute name="VALUE" x="33.909" y="-2.292" size="1.27" layer="27"/>
 </element>
 <element name="J7" library="MCP" package="KK-156-5" value="KK-156-5" x="60.96" y="5.08" smashed="yes" rot="R180">
 <attribute name="NAME" x="53.721" y="8.134" size="1.27" layer="25"/>
-<attribute name="VALUE" x="49.27" y="9.525" size="1.27" layer="27" rot="R270"/>
+<attribute name="VALUE" x="58.039" y="-2.038" size="1.27" layer="27"/>
 </element>
 <element name="J8" library="MCP" package="MSTBV2" value="MSTB-02" x="3.81" y="62.23" smashed="yes" rot="R90">
@@
 <element name="JP9" library="MCP" package="1X02_LOCK" value="NCEPWR" x="19.304" y="24.384" smashed="yes" rot="R270">
 <attribute name="NAME" x="16.5608" y="23.6982" size="0.8128" layer="25" ratio="10" rot="R270"/>
-<attribute name="VALUE" x="22.606" y="19.177" size="1.27" layer="48" rot="R180"/>
+<attribute name="VALUE" x="21.844" y="18.415" size="1.27" layer="48" rot="R180"/>
 </element>
 <element name="SV2" library="con-lsta" package="FE15" value="929850-01-15" x="41.91" y="57.15" smashed="yes" rot="R180">
@@
 </element>
 <element name="F1" library="SparkFun" package="PTC" value="PTCPTH" x="33.274" y="16.764"/>
+<element name="U$2" library="SparkFun" package="OSHW-LOGO-M" value="OSHW-LOGOM" x="20.066" y="6.096" smashed="yes"/>
 </elements>
 <signals>
