File: RailroadShield.sch (EAGLE design)
At the start: 70 parts, among them J1 RJ12, J2 RJ12, J3 RJ12, J4 RJ45, J5 RJ45, J6 5-pin molex, J7 5-pin Molex, J9 .200 2-pin, Q2 BC817-16LT1G, U1 LM393M, U2 MCP2515-SO, U3 MCP2551-SN, U4 MAX3468CSA, U5 MAX3468CSA, U6 MAX3468CSA, U7 LM317LM, U8 6N137, Y1 16Mhz

Commit message: 2.2
Parts:
- removed C7: .1uF, SparkFun:CAP0402-CAP
- removed J9: .200 2-pin, con-phoenix-500:MSTBV2
- removed MOD1: ARDUINO DUEMILANOVE, microbuilder:ARDUINODUEMILANOVE
- removed Q2: BC817-16LT1G, SparkFun:TRANSISTOR_NPNSOT23-3
- added C4: 0.01uf, MCP:CAP0805
- added J8: MSTB-02, MCP:MSTBV2
- added Q1: PMBT2222, MCP:TRANSISTOR_NPNSOT23-3
- added U$1: ARDUINODUEMILANOVE, MCP:ARDUINODUEMILANOVE
- C1, C2, C3: value .1uf -> 0.01uf; device SparkFun:CAP0402-CAP -> MCP:CAP0805
- C5, C6: value .1uF -> 0.01uf; device SparkFun:CAP0402-CAP -> MCP:CAP0805
- D1, D2: value (none) -> 1N4448WT; device SparkFun:DIODESOT23 -> MCP:DIODESOD
- J1, J2, J3: value RJ12 -> 5520250-3; device con-amp:520250-3 -> MCP:RJ11-6X
- J4, J5: value RJ45 -> 5520426-4; device con-tycoelectronics:RJ45-8X -> MCP:RJ45-8X
- J6: value 5-pin molex -> KK-156-5; device con-molex:KK-156-5 -> MCP:KK-156-5
- J7: value 5-pin Molex -> KK-156-5; device con-molex:KK-156-5 -> MCP:KK-156-5
- JP1: value LN_TERM -> LN-TERM; device SparkFun:JUMPER-2PTH -> MCP:JUMPER-2PTH_LOCK
- JP2: device SparkFun:JUMPER-3PTH -> MCP:JUMPER-3PTH
- JP3: value CAN-INT -> RxD; device SparkFun:JUMPER-2PTH -> MCP:JUMPER-3PTH
- JP4: value TXD -> EN; device SparkFun:JUMPER-2PTH -> MCP:JUMPER-3PTH
- JP5: value RXD -> TxD; device SparkFun:JUMPER-3PTH -> MCP:JUMPER-3PTH
- JP6: value EN -> MA04-2; device SparkFun:JUMPER-3PTH -> MCP:MA04-2
- JP7: value TXD -> LNTX; device SparkFun:JUMPER-3PTH -> MCP:JUMPER-2PTH_LOCK
- JP8: value CAN-CS -> CANPWR; device SparkFun:JUMPER-2PTH -> MCP:JUMPER-2PTH_LOCK
- JP9: value (none) -> NCEPWR; device con-lstb:MA04-2 -> MCP:JUMPER-2PTH_LOCK
- LED3, LED4: value Red -> Green
- R1, R10, R11, R13, R3, R4, R5, R6, R7, R8: device rcl:R-US_R0402 -> rcl:R-US_R0805
- R12: device SparkFun:RESISTOR0402-RES -> rcl:R-US_R0805
- R14: value 1K -> 1k; device SparkFun:RESISTOR0402-RES -> rcl:R-US_R0805
- R15, R16, R17, R18, R19, R20, R21, R22: value 680R -> 660R; device rcl:R-US_R0402 -> MCP:RESISTOR
- R2: value 15R -> 18R; device rcl:R-US_R0402 -> rcl:R-US_R0805
- R9: value 1K -> 1k; device rcl:R-US_R0402 -> rcl:R-US_R0805
- S1, S2, S3, S4: value 611-PTS645SH70LFS -> B3F-1052; device switch-omron:10-XX -> MCP:10-XX
- S5: value (none) -> B3F-1000; device switch-omron:10-XX -> MCP:10-XX
- U2: value MCP2515-SO -> MCP2515-ST; device MCP:MCP2515-SO -> MCP:MCP2515-ST
- U4, U5, U6: device maxim:MAX3468CSA -> MCP:MAX3468CSA
- U7: value LM317LM -> LM317LCDR; device linear:LM317LD -> MCP:LM317LD
- U8: value 6N137 -> 6N137SD; device optocoupler:6N137 -> MCP:6N137S
- Y1: device SparkFun:RESONATORPTH -> MCP:RESONATORPTH
Connections:
- net +IN renamed N$10
- net +OUT renamed N$8
- net -IN renamed N$9
- net -OUT renamed N$7
- net L1+ renamed N$5
- net L2+ renamed N$2
- net L3+ renamed N$3
- net L4+ renamed N$4
- net OSC1 renamed N$12
- net OSC2 renamed N$13
- net SHIELD renamed N$6
- removed net CAN-CS: JP8.1, U2./CS
- removed net CAN-INT: JP3.1, U2./INT
- removed net DCCA: J9-1.SK, R14.1
- new net N$11: J8-1.SK, R14.1
- new net N$14: D2.A, JP9.1
- new net N$15: D1.A, JP8.1
- net A/RESET: now also U$1./RESET; no longer MOD1./RESET
- net CMRIRX: now also JP3.1; no longer JP5.1
- net CMRITX: now also JP5.1; no longer JP7.1
- net CMRITXEN: now also JP4.1; no longer JP6.1
- net D0: now also JP3.2, U$1.D0; no longer JP5.2, MOD1.D0
- net D1: now also JP5.2, U$1.D1; no longer JP7.2, MOD1.D1
- net D10: now also JP6.7, U$1.D10; no longer JP9.4, MOD1.D10
- net D11: now also U$1.D11; no longer MOD1.D11
- net D12: now also U$1.D12; no longer MOD1.D12
- net D13: now also U$1.D13; no longer MOD1.D13
- net D2: now also JP6.1, U$1.D2; no longer JP9.6, MOD1.D2
- net D3: now also U$1.D3, U2./INT; no longer JP3.2, MOD1.D3
- net D4: now also JP6.3, U$1.D4; no longer JP9.2, MOD1.D4
- net D5: now also JP4.2, U$1.D5; no longer JP6.2, MOD1.D5
- net D6: now also JP6.5, U$1.D6; no longer JP9.8, MOD1.D6
- net D7: now also JP7.2, U$1.D7; no longer JP4.1, MOD1.D7
- net D8: now also U$1.D8; no longer MOD1.D8
- net D9: now also U$1.D9, U2./CS; no longer JP8.2, MOD1.D9
- net DCCB: now also J8-2.SK; no longer J9-2.SK
- net GND: now also C4.2, U$1.GND, U$1.GND1, U$1.GND2; no longer C7.2, MOD1.GND, MOD1.GND1, MOD1.GND2
- net IO1: now also JP6.2; no longer JP9.7
- net IO2: now also JP6.4; no longer JP9.5
- net IO3: now also JP6.6; no longer JP9.3
- net IO4: now also JP6.8; no longer JP9.1
- net LN-TX: now also Q1.B; no longer Q2.B
- net LNTX: now also JP7.1; no longer JP4.2
- net LOCONET: now also Q1.C; no longer Q2.C
- net N$1: now also Q1.E; no longer Q2.E
- net NCERX: now also JP3.3; no longer JP5.3
- net NCETX: now also JP5.3; no longer JP7.3
- net NCETXEN: now also JP4.3; no longer JP6.3
- net V+: now also JP8.2, JP9.2, U$1.VIN; no longer D1.A, D2.A, MOD1.VIN
- net VCC: now also C4.1, U$1.5V; no longer C7.1, MOD1.5V
Other:
- note added: "2.2"
- note added: "Locoduino/RailroadShield/"
- note removed: "2.1smd"
- note removed: "Locoduino/RailroadShield/2.0/"
- moved on the sheet: C1, C2, C3, C5, C6, D2, J1, J2, J3, JP1, JP5, JP8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

Commit message: 2.3
Parts:
- removed JP3: RxD, MCP:JUMPER-3PTH
- removed JP4: EN, MCP:JUMPER-3PTH
- removed JP5: TxD, MCP:JUMPER-3PTH
- removed JP6: MA04-2, MCP:MA04-2
- removed JP7: LNTX, MCP:JUMPER-2PTH_LOCK
- removed R15, R16, R17, R18, R19, R20, R21, R22: 660R, MCP:RESISTOR
- added RN1: 660R, resistor-sil:G04R
- added RN2: 660R, resistor-sil:E4R
- added SV1, SV2: (no value), con-lsta:FE15-1
- D1, D2: device MCP:DIODESOD -> MCP:DIODESOT23
- J1, J2, J3: device MCP:RJ11-6X -> MCP:RJ11-6XRA
- JP2: value RXD-LN -> ShieldGnd; device MCP:JUMPER-3PTH -> MCP:JUMPER-2PTH_LOCK
- U2: value MCP2515-ST -> MCP2515-SO; device MCP:MCP2515-ST -> MCP:MCP2515-SO
Connections:
- net D11 renamed MOSI
- net D12 renamed MISO
- net D13 renamed SCK
- removed net S1+: R19.1, S1.P, S1.P1
- removed net S2+: R20.1, S2.P, S2.P1
- removed net S3+: R21.1, S3.P, S3.P1
- removed net S4+: R22.1, S4.P, S4.P1
- new net A0: SV2.12, U$1.A0
- new net A1: SV2.13, U$1.A1
- new net A2: SV2.14, U$1.A2
- new net A3: SV2.15, U$1.A3
- new net CANCS: SV1.11, U2./CS
- new net CANINT: SV1.10, U2./INT
- new net N$16: RN2A.2, S1.P
- new net N$17: RN2B.2, S2.P
- new net N$18: RN2C.2, S3.P
- new net N$19: RN2D.2, S4.P
- net CMRIRX: now also SV1.1; no longer JP3.1
- net CMRITX: now also SV1.2; no longer JP5.1
- net CMRITXEN: now also SV1.3; no longer JP4.1
- net D0: now also SV2.1; no longer JP3.2
- net D1: now also SV2.2; no longer JP5.2
- net D10: now also SV2.11; no longer JP6.7
- net D2: now also SV2.3; no longer JP6.1
- net D3: now also SV2.4; no longer U2./INT
- net D4: now also SV2.5; no longer JP6.3
- net D5: now also SV2.6; no longer JP4.2
- net D6: now also SV2.7; no longer JP6.5
- net D7: now also SV2.8; no longer JP7.2
- net D8: now also SV2.9; no longer JP2.2
- net D9: now also SV2.10; no longer U2./CS
- net DCCRX: now also SV1.9; no longer JP2.1
- net GND: now also JP2.1; no longer S1.S1, S2.S1, S3.S1, S4.S1
- net IO1: now also RN2A.1, SV1.15; no longer JP6.2, R19.2
- net IO2: now also RN2B.1, SV1.14; no longer JP6.4, R20.2
- net IO3: now also RN2C.1, SV1.13; no longer JP6.6, R21.2
- net IO4: now also RN2D.1, SV1.12; no longer JP6.8, R22.2
- net LNRX: now also SV1.7; no longer JP2.3
- net LNTX: now also SV1.8; no longer JP7.1
- net N$2: now also LED1.A, RN1.2; no longer LED2.A, R16.1
- net N$3: now also LED2.A, RN1.3; no longer LED3.A, R17.1
- net N$4: now also LED3.A, RN1.4; no longer LED4.A, R18.1
- net N$5: now also LED4.A, RN1.5; no longer LED1.A, R15.1
- net N$6: now also JP2.2
- net NCERX: now also SV1.4; no longer JP3.3
- net NCETX: now also SV1.5; no longer JP5.3
- net NCETXEN: now also SV1.6; no longer JP4.3
- net VCC: now also RN1.1; no longer R15.2, R16.2, R17.2, R18.2
Other:
- note added: "2.3"
- note added: "I2C"
- note removed: "2.2"
- note removed: "I/O Test points"
- note removed: "MISO"
- note removed: "MOSI"
- note removed: "RX"
- note removed: "SCK"
- note removed: "TX"
- note removed: "TXEN"
- moved on the sheet: C1, C2, C3, C4, C5, C6, J8-1, J8-2, LED1, LED2, LED3, LED4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
