File: RailroadShield.sch (EAGLE design)
At the start: 61 parts, among them J1 5520250-3, J2 5520250-3, J3 5520250-3, J4 5520426-4, J5 5520426-4, J6 KK-156-5, J7 KK-156-5, J8 MSTB-02, Q1 PMBT2222, U1 LM393M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

Commit message: 2.4
Parts:
- added F1: PTCPTH, SparkFun:PTCPTH
- D1, D2: value 1N4448WT -> BAV199; device MCP:DIODESOT23 -> diode:BAV199
- JP2: value ShieldGnd -> CMRI Shield
- LED5: value DCC -> Yellow
- LED6: value Loconet -> Blue
- SV1, SV2: value (none) -> 929850-01-15
- Y1: value 16Mhz -> 16Mhz 81-CSTLS16M0X53-B0
Connections:
- removed net TERM-PWR: JP1.1, U7.VI
- new net N$20: JP1.2, R10.2, U7.ADJ
- new net N$21: F1.2, U$1.VIN
- net CAN-PWR+: now also D1.AC; no longer D1.C
- net LOCONET: now also JP1.1; no longer R10.2, U7.ADJ
- net NCE-PWR+: now also D2.AC; no longer D2.C
- net V+: now also F1.1, U7.VI; no longer JP1.2, U$1.VIN
Other:
- note added: "2.4"
- note removed: "2.3"
- moved on the sheet: JP1, JP8, JP9, Q1, R1, R10, R2, U7
